File: design pcb.kicad_pcb (KiCad board)
At the start: 2 copper layers, 0 parts

Commit message: v2
Routing:
- net (no net): track 3090.9 -> 50.9 mm, vias 131 -> 96
- removed copper zone on F.Cu, net GND

Commit message: v3
Routing:
- net (no net): track 50.9 -> 2891.1 mm, vias 96 -> 131
- added copper zone on F.Cu, net GND
- removed copper zone on F.Cu, net (none)

Commit message: v4
Routing:
- net (no net): track 2891.1 -> 2551.8 mm, vias 131 -> 130
- added copper zone on F.Cu, net 5V
