File: design pcb.kicad_pcb (KiCad board)
At the start: 2 copper layers, 0 parts

Commit message: v6
Routing:
- removed copper zone on F.Cu, net GND
Other:
- board outline added: 155 x 120 mm

Commit message: v7
Routing:
- net (no net): track 2552.2 -> 2123.7 mm, vias 130 -> 87
- net GND: track 0.00 -> 290.9 mm, vias 0 -> 41
- added copper zone on F.Cu, net GND
- added copper zone on F.Cu, net trash
- removed copper zone on F.Cu, net 5V
Other:
- board size 155 x 120 mm -> 140 x 120 mm

Commit message: v8
Routing:
- net GND: track 290.9 -> 290.2 mm

Commit message: v9
Routing:
- net (no net): track 2123.7 -> 2289.3 mm, vias 87 -> 84
- net GND: track 290.2 -> 387.0 mm, vias 41 -> 43

Commit message: v9
Routing:
- net (no net): track 2289.3 -> 2356.5 mm, vias 84 -> 85
- net GND: track 387.0 -> 382.1 mm, vias 43 -> 42
